File: Sensor.sch (KiCad schematic (older format))
At the start: 5 parts

Commit message: Schematic and component value worksheet
Parts:
- removed C?: 10uF, ~, symbol C
- removed R?: 1K, ~, symbol R
- added C? (x8): Cfilter, ~, symbol C
- added P?: CONN_12, symbol CONN_12
- added R?: FloorRef1, ~, symbol R
- added R?: FloorRef2, ~, symbol R
- added R? (x16): OpR1, ~, symbol R
- added R? (x16): OpR2, ~, symbol R
- added R? (x7): RD, ~, symbol R
- added R? (x8): Rfilter, ~, symbol R
- added TH? (x7): THERM, ~, symbol THERMISTOR
- added U? (x8): LM324, symbol LM324
- R?: value 330 1% -> RD
- TH?: value THERMISTOR 330 -> THERM
Connections:
- net labels added: ARef, Control, Out1, Out2, Out3, Out4, Out5, Out6, Out7, Out8, Sense1, Sense2, Sense3, Sense4, Sense5, Sense6, Sense7, Sense8, Vcc, Vpower
- net labels removed: +5V, AGND
- wire segments 12 -> 179
Other:
- note added: "Amp Array"
- note added: "Sensor Array"
- note removed: "Output"
- note removed: "uC Power Control"
- moved on the sheet: Q?, R?, TH?

Commit message: Update With Schematic PDF
Parts:
- added 10uF: C, ~, symbol C
Connections:
- net ARef: now also 10uF.2
- net GND: now also 10uF.1
Changed lines of the file:
@@
 Sheet 1 1
 Title ""
-Date "6 dec 2014"
+Date "8 dec 2014"
 Rev ""
 Comp ""
@@
 Wire Wire Line
 	8550 6300 8650 6300
+$Comp
+L C 10uF
+U 1 1 548508E8
+P 9600 2350
+F 0 "10uF" H 9600 2450 40  0000 L CNN
+F 1 "C" H 9606 2265 40  0000 L CNN
+F 2 "~" H 9638 2200 30  0000 C CNN
+F 3 "~" H 9600 2350 60  0000 C CNN
+	1    9600 2350
+	0    1    1    0
+$EndComp
+Wire Wire Line
+	9400 2350 9200 2350
+Connection ~ 9200 2350
+Wire Wire Line
+	9800 2350 9850 2350
+Wire Wire Line
+	9850 2350 9850 2500
+$Comp
+L GND #PWR?
+U 1 1 54850A98
+P 9850 2500
+F 0 "#PWR?" H 9850 2500 30  0001 C CNN
+F 1 "GND" H 9850 2430 30  0001 C CNN
+F 2 "" H 9850 2500 60  0000 C CNN
+F 3 "" H 9850 2500 60  0000 C CNN
+	1    9850 2500
+	1    0    0    -1
+$EndComp
 $EndSCHEMATC

Commit message: Layout Partial
Schematic Finished and Layout partially done
Parts:
- removed C? (x7): Cfilter, ~, symbol C
- removed Q?: MOS_N, ~, symbol MOS_N
- removed R? (x15): OpR2, ~, symbol R
- removed R? (x15): OpR1, ~, symbol R
- removed R? (x7): RD, ~, symbol R
- removed R? (x7): Rfilter, ~, symbol R
- removed TH? (x7): THERM, ~, symbol THERMISTOR
- removed U? (x7): LM324, symbol LM324
- added C1, C2, C3, C5, C6, C7, C8: Cfilter, ~, symbol C
- added C10, C11, C12, C13, C9: Cdecouple, ~, symbol C
- added Q1: MOS_P, ~, symbol MOS_P
- added R10, R11, R12, R13, R14, R16, R31, R32, R33, R34, R35, R36, R37, R38, R9: OpR1, ~, symbol R
- added R17, R18, R19, R20, R21, R22, R23, R39, R40, R41, R42, R43, R44, R45, R46: OpR2, ~, symbol R
- added R2, R3, R4, R5, R6, R7, R8: RD, ~, symbol R
- added R25, R26, R27, R47, R48, R49, R50: Rfilter, ~, symbol R
- added R51: 10K, ~, symbol R
- added TH2, TH3, TH4, TH5, TH6, TH7, TH8: THERM, ~, symbol THERMISTOR
- added U1, U2, U5: LM324, symbol LM324
- added unit 1 of U3
- added unit 2 of U3
- added unit 3 of U3
- added U4: TL071, symbol TL071
- C14: renamed from 10uF; value C -> 10uF
- gave numbers to parts that had none: 10
Connections:
- net ARef: now also Q1.D, R2.1, R3.1, R4.1, R5.1, R6.1, R7.1, R8.1
- net Control: now also Q1.G, R51.1
- net GND: now also U3.11 (V-), C1.2, C10.2, C11.2, C12.2, C13.2, C2.2, C3.2, C5.2, C6.2, C7.2, C8.2, C9.2, R17.1, R18.1, R19.1, R20.1, R39.1, R40.1, R41.1, R42.1, R51.2, TH2.2, TH3.2, TH4.2, TH5.2, TH6.2, TH7.2, TH8.2, U1.11 (V-), U1.11 (V-), U1.11 (V-), U1.11 (V-), U2.11 (V-), U2.11 (V-), U2.11 (V-), U2.11 (V-), U3.11 (V-), U3.11 (V-), U3.11 (V-), U4.4 (V-), U5.11 (V-), U5.11 (V-), U5.11 (V-), U5.11 (V-); no longer U3.4 (V+)
- net Out2: now also R25.1
- net Out3: now also R26.1
- net Out4: now also R27.1
- net Out5: now also R50.1
- net Out6: now also R47.1
- net Out7: now also R48.1
- net Out8: now also R49.1
- net Sense1: now also U1.1, U1.2 (-); no longer R1.2, TH1.1
- net Sense2: now also R9.2, U1.6 (-), U1.7
- net Sense3: now also R11.2, U1.8, U1.9 (-)
- net Sense4: now also R13.2, U1.13 (-), U1.14
- net Sense5: now also R37.2, U2.1, U2.2 (-)
- net Sense6: now also R31.2, U2.6 (-), U2.7
- net Sense7: now also R33.2, U2.8, U2.9 (-)
- net Sense8: now also R35.2, U2.13 (-), U2.14
- net Vcc: now also U3.4 (V+), C10.1, C11.1, C12.1, C13.1, C9.1, U1.4 (V+), U1.4 (V+), U1.4 (V+), U1.4 (V+), U2.4 (V+), U2.4 (V+), U2.4 (V+), U2.4 (V+), U3.4 (V+), U3.4 (V+), U3.4 (V+), U4.7 (V+), U5.4 (V+), U5.4 (V+), U5.4 (V+), U5.4 (V+); no longer U3.11 (V-)
- net Vpower: now also Q1.S
- net at R29.2, R30.1: now also U4.3 (+)
- net at R24.1, R28.2: now also U3.14; no longer U3.1
- net at R15.1, R24.2: now also U3.12 (+); no longer U3.3 (+)
- new net: R1.2, TH1.1, U1.3 (+)
- new net: R16.1, R20.2, U3.13 (-)
- new net: R2.2, TH2.1, U1.5 (+)
- new net: R3.2, TH3.1, U1.10 (+)
- new net: R4.2, TH4.1, U1.12 (+)
- new net: R5.2, TH5.1, U2.3 (+)
- new net: R6.2, TH6.1, U2.5 (+)
- new net: R7.2, TH7.1, U2.10 (+)
- new net: R8.2, TH8.1, U2.12 (+)
- new net: R21.1, R25.2, U3.1
- new net: R10.1, R17.2, U3.2 (-)
- new net: R21.2, R9.1, U3.3 (+)
- new net: R11.1, R22.2, U3.5 (+)
- new net: R12.1, R18.2, U3.6 (-)
- new net: R22.1, R26.2, U3.7
- new net: R13.1, R23.2, U3.10 (+)
- new net: R23.1, R27.2, U3.8
- new net: R14.1, R19.2, U3.9 (-)
- new net: R37.1, R46.2, U5.12 (+)
- new net: R38.1, R42.2, U5.13 (-)
- new net: R46.1, R50.2, U5.14
- new net: R43.1, R47.2, U5.1
- new net: R32.1, R39.2, U5.2 (-)
- new net: R31.1, R43.2, U5.3 (+)
- new net: R33.1, R44.2, U5.5 (+)
- new net: R34.1, R40.2, U5.6 (-)
- new net: R44.1, R48.2, U5.7
- new net: R35.1, R45.2, U5.10 (+)
- new net: R45.1, R49.2, U5.8
- new net: R36.1, R41.2, U5.9 (-)
- new net Vmin: R10.2, R12.2, R14.2, R16.2, R32.2, R34.2, R36.2, R38.2, U4.2 (-), U4.6
Other:
- note added: "OpAmp IC decouples"
- moved on the sheet: C14, C4, P1, R15, R24, R28, R29, R30

Commit message: Updates
Closer to final layout
Parts:
- Q1: footprint ~ -> SOT23
Changed lines of the file:
@@
 Sheet 1 1
 Title ""
-Date "13 dec 2014"
+Date "17 dec 2014"
 Rev ""
 Comp ""
@@
 F 0 "Q1" H 6700 9040 60  0000 R CNN
 F 1 "MOS_P" H 6700 8670 60  0000 R CNN
-F 2 "~" H 6700 8850 60  0000 C CNN
+F 2 "SOT23" H 6700 8850 60  0000 C CNN
 F 3 "~" H 6700 8850 60  0000 C CNN
 	1    6700 8850
