File: TrinketWind.kicad_pcb (KiCad board)
At the start: 2 copper layers, 80 parts, among them P1 CONN_12, Q1 MOS_P, U1 LM324, U2 LM324, U3 LM324, U4 TL071, U5 LM324

Commit message: Updates
Closer to final layout
Parts:
- C10, C14, C9, Q1, R12, R18, R22, R29, R30, R51, U4: moved to B.Cu
- moved R29 144.5 mm to (49.4, 201.0), turned to 90 degrees
- moved R51 142.6 mm to (64.4, 200.4), turned to 90 degrees
- moved R30 141.7 mm to (49.4, 198.2), turned to 90 degrees
- moved U4 141.4 mm to (52.8, 198.4), turned to 270 degrees
- moved Q1 141.2 mm to (58.8, 198.8), turned to 180 degrees
- moved C14 140.9 mm to (62.2, 198.6), turned to 90 degrees
- moved R22 126.9 mm to (57.0, 184.3), turned to 270 degrees
- moved R18 124.1 mm to (53.2, 181.0), turned to 270 degrees
- moved R12 123.9 mm to (55.0, 181.0), turned to 90 degrees
- moved C10 113.1 mm to (49.8, 169.4), turned to 180 degrees
- moved C9 110.0 mm to (66.5, 167.9), turned to 90 degrees
- moved R43 5.50 mm to (61.0, 184.0), turned to 270 degrees
- moved R11 4.05 mm to (56.8, 181.0), turned to 90 degrees
- moved R31 3.44 mm to (61.2, 180.7)
- moved R10 2.44 mm to (48.4, 181.0)
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Connections:
- U4 pad 1: (no net) -> Vmin
- U4 pad 2: Vmin -> Vcc
- U4 pad 4: GND -> Vmin
- U4 pad 5: (no net) -> GND
Routing:
- net GND: track 26.8 -> 223.1 mm, vias 2 -> 14
- net ARef: track 53.0 -> 160.1 mm, vias 2 -> 5
- net Vcc: track 0.00 -> 90.1 mm, vias 0 -> 6
- net Vmin: track 0.00 -> 79.4 mm, vias 0 -> 5
- net Sense8: track 1.27 -> 32.3 mm
- net Sense1: track 1.27 -> 29.2 mm, vias 0 -> 2
- net Sense5: track 1.27 -> 28.8 mm
- net Sense4: track 1.27 -> 26.9 mm, vias 0 -> 2
- net Sense2: track 1.27 -> 16.9 mm
- net Sense6: track 1.27 -> 15.3 mm, vias 0 -> 2
- net N-000008: track 0.00 -> 10.4 mm
- net N-0000024: track 0.00 -> 6.36 mm
- net N-0000062: track 22.5 -> 27.8 mm
- net N-0000060: track 32.7 -> 28.4 mm, vias 1 -> 3
- net N-0000010: track 0.00 -> 3.99 mm
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Other:
- net class HiCurrent added: clearance 0.254, trace_width 0.762, via_dia 1.143, via_drill 0.889

Commit message: 12-17-14
Parts:
- C11, C12, C13, R25, R26, R27, R28, R47, R48, R49, R50: moved to B.Cu
- moved C4 190.7 mm to (213.5, 182.2), turned to 270 degrees
- moved C1 188.8 mm to (211.0, 182.2), turned to 270 degrees
- moved R28 187.1 mm to (213.5, 176.7), turned to 90 degrees
- moved C2 186.9 mm to (208.4, 182.2), turned to 270 degrees
- moved R25 185.2 mm to (211.1, 176.7), turned to 90 degrees
- moved C3 185.0 mm to (205.9, 182.2), turned to 270 degrees
- moved R26 183.2 mm to (208.4, 176.7), turned to 90 degrees
- moved C8 183.2 mm to (203.4, 182.2), turned to 270 degrees
- moved R27 181.3 mm to (205.9, 176.7), turned to 90 degrees
- moved C5 181.3 mm to (200.8, 182.2), turned to 270 degrees
- moved C6 179.4 mm to (198.3, 182.2), turned to 270 degrees
- moved R50 179.4 mm to (203.4, 176.7), turned to 90 degrees
- moved C7 177.6 mm to (195.8, 182.2), turned to 270 degrees
- moved R47 177.6 mm to (200.8, 176.7), turned to 90 degrees
- moved R48 175.7 mm to (198.3, 176.8), turned to 90 degrees
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Connections:
- C1 pad 1: (no net) -> Out2
- C2 pad 1: (no net) -> Out3
- C3 pad 1: (no net) -> Out4
- C4 pad 1: (no net) -> Out1
- C5 pad 1: (no net) -> Out6
- C6 pad 1: (no net) -> Out7
- C7 pad 1: (no net) -> Out8
- C8 pad 1: (no net) -> Out5
Routing:
- net GND: track 223.1 -> 355.3 mm, vias 14 -> 17
- net N-0000021: track 1.76 -> 58.6 mm, vias 0 -> 2
- net N-0000055: track 2.38 -> 47.3 mm
- net N-0000039: track 1.51 -> 44.2 mm, vias 0 -> 2
- net Vcc: track 90.1 -> 130.9 mm
- net N-0000030: track 2.32 -> 42.3 mm, vias 0 -> 4
- net N-0000045: track 1.72 -> 39.9 mm, vias 0 -> 4
- net N-000009: track 1.62 -> 38.1 mm, vias 0 -> 2
- net N-0000014: track 2.38 -> 36.7 mm, vias 0 -> 2
- net N-000003: track 2.32 -> 32.9 mm, vias 0 -> 2
- net Control: track 0.00 -> 23.7 mm, vias 0 -> 2
- net Vpower: track 0.00 -> 21.1 mm, vias 0 -> 2
- net Vmin: track 79.4 -> 90.6 mm, vias 5 -> 7
- net Sense2: track 16.9 -> 22.6 mm
- net N-000006: track 14.6 -> 9.84 mm
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Other:
- board outline added: 31.3 x 77.7 mm

Commit message: Final?
Parts:
- added 1PIN: P***, 1pin, F.Cu at (210.8, 116.0)
- added 1PIN: P***, 1pin, F.Cu at (187.4, 115.9)
Routing:
- net GND: track 355.3 -> 361.7 mm
- net (no net): vias 0 -> 1
- added copper zone on B.Cu, net GND
- added copper zone on F.Cu, net GND
Other:
- board text added: "KRATZ INDUSTRIES 12/18/2014"
